File: pcb/slam.kicad_pcb (KiCad board)
At the start: 4 copper layers, 40.7 x 40.9 mm, 64 parts, among them J1 Conn_01x02_Pin, J10 Conn_01x06_Socket, J11 Conn_01x08_Pin, J2 Conn_02x02_Odd_Even, J3 USB_C_Receptacle_USB2.0_16P, J4 Conn_01x02_Pin, J5 Conn_01x02_Pin, J6 Conn_01x02_Pin, J7 Conn_01x02_Pin, J8 Conn_01x02_Pin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

Commit message: update diode, usb routing
Parts:
- D2: value 1N4148 -> 1N5819WS; footprint Diode_SMD:D_SOD-323_HandSoldering -> Diode_SMD:D_SOD-123
- moved D2 3.86 mm to (94.3, 109.2)
Routing:
- net +5V: track 18.6 -> 21.1 mm
- net /Motors/LIDAR_OUT2: track 5.36 -> 7.40 mm
- net GND: vias 64 -> 63
