File: pcb/motors.kicad_sch (KiCad schematic)
At the start: 21 parts, among them J4 Conn_01x02_Pin, J5 Conn_01x02_Pin, J6 Conn_01x02_Pin, J7 Conn_01x02_Pin, J8 Conn_01x02_Pin, Q1 AO3400A, U3 DRV8833PWP, U4 DRV8833PWP

Commit message: cleanup pcb
Connections:
- net LIDAR_IN: no longer R8.1
- net at Q1.1 (G), R7.2: now also R8.1
Other:
- moved on the sheet: R8
Changed lines of the file:
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@@
+	)
+	(junction
+		(at 128.27 72.39)
+		(diameter 0)
+		(color 0 0 0 0)
+	)
+	(junction
+		(at 135.89 67.31)
+		(diameter 0)
+		(color 0 0 0 0)
+	)
+	(junction
+		(at 30.48 106.68)
+		(diameter 0)
+		(color 0 0 0 0)
 	)
 	(junction
@@
 	)
 	(junction
-		(at 135.89 67.31)
-		(diameter 0)
-		(color 0 0 0 0)
-	)
-	(junction
-		(at 30.48 106.68)
-		(diameter 0)
-		(color 0 0 0 0)
-	)
-	(junction
 		(at 128.27 39.37)
 		(diameter 0)
@@
 	(wire
 		(pts
-			(xy 129.54 78.74) (xy 135.89 78.74)
-		)
-		(stroke
-			(width 0)
-			(type default)
-		)
-	)
-	(wire
-		(pts
 			(xy 30.48 106.68) (xy 30.48 107.95)
 		)
@@
 	(wire
 		(pts
-			(xy 120.65 72.39) (xy 120.65 78.74)
-		)
-		(stroke
-			(width 0)
-			(type default)
-		)
-	)
-	(wire
-		(pts
 			(xy 67.31 33.02) (xy 69.85 33.02)
 		)
@@
 	(wire
 		(pts
-			(xy 120.65 78.74) (xy 121.92 78.74)
-		)
-		(stroke
-			(width 0)
-			(type default)
-		)
-	)
-	(wire
-		(pts
 			(xy 135.89 78.74) (xy 135.89 82.55)
 		)
@@
 		(pts
 			(xy 69.85 33.02) (xy 69.85 36.83)
+		)
+		(stroke
+			(width 0)
+			(type default)
+		)
+	)
+	(wire
+		(pts
+			(xy 128.27 72.39) (xy 128.27 78.74)
 		)
 		(stroke
@@
 	(symbol
 		(lib_id "Device:R")
-		(at 125.73 78.74 90)
+		(at 132.08 78.74 90)
 		(mirror x)
 		(unit 1)
@@
 		(dnp no)
 		(property "Reference" "R8"
-			(at 125.73 85.09 90)
+			(at 132.08 85.09 90)
 			(show_name no)
 			(do_not_autoplace no)
@@
 		)
 		(property "Value" "10k"
-			(at 125.73 82.55 90)
+			(at 132.08 82.55 90)
 			(show_name no)
 			(do_not_autoplace no)
@@
 		)
 		(property "Footprint" "Resistor_SMD:R_0805_2012Metric_Pad1.20x1.40mm_HandSolder"
-			(at 125.73 76.962 90)
+			(at 132.08 76.962 90)
 			(hide yes)
 			(show_name no)
@@
 		)
 		(property "Datasheet" ""
-			(at 125.73 78.74 0)
+			(at 132.08 78.74 0)
 			(hide yes)
 			(show_name no)
@@
 		)
 		(property "Description" "Resistor"
-			(at 125.73 78.74 0)
+			(at 132.08 78.74 0)
 			(hide yes)
 			(show_name no)
@@
 		)
 		(property "LCSC" "C2930231"
-			(at 125.73 78.74 90)
+			(at 132.08 78.74 90)
 			(hide yes)
 			(show_name no)
@@
 		)
 		(property "KLC_S3.3" ""
-			(at 125.73 78.74 90)
+			(at 132.08 78.74 90)
 			(hide yes)
 			(show_name no)
@@
 		)
 		(property "KLC_S4.1" ""
-			(at 125.73 78.74 90)
+			(at 132.08 78.74 90)
 			(hide yes)
 			(show_name no)
