File: pcb/slam.kicad_sch (KiCad schematic)
At the start: 28 parts, among them J1 Conn_01x02_Pin, J2 Conn_02x02_Odd_Even, J3 USB_C_Receptacle_USB2.0_16P, SW1 SW_Push, SW2 SW_Push, U1 STM32F401RETx, U2 TLV1117-33, Y1 25 MHz

Commit message: pcb: fix boot button and some traces
Connections:
- net +3.3V is gone; now on net +3V3: SW1.1
